Commit message: commit1

File: src/car/urdf/localization-robot/robot.xacro (robot description, xacro)
@@ -1,5 +1,5 @@
 <?xml version="1.0"?>
 <robot name="simple_robot" xmlns:xacro="http://www.ros.org/wiki/xacro">
-        <xacro:include filename="$(find car)/model/slam-robot/gazebo.xacro"/>
+        <xacro:include filename="$(find car)/urdf/localization-robot/gazebo.xacro"/>
         <link name="base_footprint"/>
         <material name="blue">

File: src/car/urdf/slam-robot/gazebo.xacro (robot description, xacro)
@@ -50,5 +50,9 @@
         <minDepth>0.001</minDepth>
         <maxVel>0.1</maxVel>
-        <material>Gazebo/Blue</material>
+        <material>
+            <ambient>0.0 0.0 1.0 1</ambient>
+            <diffuse>0.0 0.0 1.0 1</diffuse>
+            <specular>0.1 0.1 0.1 1</specular>
+        </material>
     </gazebo>
     <gazebo reference="rb_link">

File: src/car/urdf/slam-robot/robot.xacro (robot description, xacro)
@@ -1,5 +1,5 @@
 <?xml version="1.0"?>
 <robot name="simple_robot" xmlns:xacro="http://www.ros.org/wiki/xacro">
-        <xacro:include filename="$(find car)/model/localization-robot/gazebo.xacro"/>
+        <xacro:include filename="$(find car)/urdf/slam-robot/gazebo.xacro"/>
         <link name="base_footprint"/>
         <material name="blue">
