Commit message: xacro Blue

File: src/car/urdf/slam-robot/gazebo.xacro (robot description, xacro)
@@ -50,9 +50,5 @@
         <minDepth>0.001</minDepth>
         <maxVel>0.1</maxVel>
-        <material>
-            <ambient>0.0 0.0 1.0 1</ambient>
-            <diffuse>0.0 0.0 1.0 1</diffuse>
-            <specular>0.1 0.1 0.1 1</specular>
-        </material>
+        <material>Gazebo/Blue</material>
     </gazebo>
     <gazebo reference="rb_link">
